Commit message: control: expanded allowed pitch rotation range from abs(80) to abs(85), added validate_fk_ik

File: control/ato_3_seg.urdf (robot description, URDF)
Before this commit: robot ato, 8 links, 7 joints
Joints:
- joint joint_1_to_bone_1: limit lower=-1.39626 upper=1.39626 effort=1.0 velocity=1.0 -> lower=-1.48353 upper=1.48353 effort=1.0 velocity=1.0
- joint joint_2_to_bone_2: limit lower=-1.39626 upper=1.39626 effort=1.0 velocity=1.0 -> lower=-1.48353 upper=1.48353 effort=1.0 velocity=1.0
- joint joint_3_to_bone_3: limit lower=-1.39626 upper=1.39626 effort=1.0 velocity=1.0 -> lower=-1.48353 upper=1.48353 effort=1.0 velocity=1.0

Commit message: control: use pytest for sanity test

File: control/ato_3_seg.urdf (robot description, URDF)
Before this commit: robot ato, 8 links, 7 joints
Joints:
- joint bone_3_to_endeffector: axis 1 0 0 -> (none)
