Commit message: control: 270 pitch range

File: ato_control/ato_3_seg.urdf (robot description, URDF)
Before this commit: robot ato, 8 links, 7 joints
Joints:
- joint joint_1_to_bone_1: limit lower=-1.48353 upper=1.48353 effort=1.0 velocity=1.0 -> lower=-2.26893 upper=2.26893 effort=1.0 velocity=1.0
- joint joint_2_to_bone_2: limit lower=-1.48353 upper=1.48353 effort=1.0 velocity=1.0 -> lower=-2.26893 upper=2.26893 effort=1.0 velocity=1.0
- joint joint_3_to_bone_3: limit lower=-1.48353 upper=1.48353 effort=1.0 velocity=1.0 -> lower=-2.26893 upper=2.26893 effort=1.0 velocity=1.0

Commit message: control: fixed issue in align_vectors and visualization

File: ato_control/ato_3_seg.urdf (robot description, URDF)
Before this commit: robot ato, 8 links, 7 joints
Joints:
- joint bone_3_to_endeffector: child endeffector -> endeffector_link

Commit message: control: evaluate_ik_cache forward_only within_reach

File: ato_control/ato_3_seg.urdf (robot description, URDF)
Before this commit: robot ato, 8 links, 7 joints
Joints:
- joint joint_1_to_bone_1: origin xyz=0 0 210 rpy=0 0 0 -> xyz=0 0 220 rpy=0 0 0
- joint joint_2_to_bone_2: origin xyz=0 0 210 rpy=0 0 0 -> xyz=0 0 220 rpy=0 0 0
- joint joint_3_to_bone_3: origin xyz=0 0 210 rpy=0 0 0 -> xyz=0 0 220 rpy=0 0 0
