Commit message: urdf: added ato_2_seg_180_deg.urdf

File: urdf/ato_3_seg_270_deg.urdf (robot description, URDF)
Before this commit: robot ato, 8 links, 7 joints
Links:
- link base_link: geometry visual mesh filename=file:///tmp/pitch_range_270/BoneAugmented_urdf_mesh.stl
- link bone_1: geometry visual mesh filename=file:///tmp/pitch_range_270/BoneAugmented_urdf_mesh.stl
- link bone_2: geometry visual mesh filename=file:///tmp/pitch_range_270/BoneAugmented_urdf_mesh.stl
- link bone_3: geometry visual mesh filename=file:///tmp/pitch_range_270/GripperDragonWithServo_urdf_mes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
- link joint_1: geometry visual mesh filename=file:///tmp/pitch_range_270/JointAugmented_urdf_mesh.stl
- link joint_2: geometry visual mesh filename=file:///tmp/pitch_range_270/JointAugmented_urdf_mesh.stl
- link joint_3: geometry visual mesh filename=file:///tmp/pitch_range_270/JointAugmented_urdf_mesh.stl
Joints:
- joint base_link_to_joint_1: limit lower=-1.5708 upper=3.14159 effort=1.0 velocity=1.0 -> lower=-2.35619 upper=2.35619 effort=1.0 velocity=1.0
- joint bone_1_to_joint_2: limit lower=-1.5708 upper=3.14159 effort=1.0 velocity=1.0 -> lower=-2.35619 upper=2.35619 effort=1.0 velocity=1.0
- joint bone_2_to_joint_3: limit lower=-1.5708 upper=3.14159 effort=1.0 velocity=1.0 -> lower=-2.35619 upper=2.35619 effort=1.0 velocity=1.0
