Commit message: refactored inverse_kinematics_pinocchio
cleaned up debugging code

updated urdf files to add dummy object for pinocchio

minor updates to env setup scripts

File: urdf/ato_2_seg_180_deg.urdf (robot description, URDF)
Before this commit: robot ato, 6 links, 5 joints
Links:
- removed link bone_2
- removed link endeffector_link
- added link dummy_object_link; visual box size=1 2 3
- added link endeffector; visual mesh filename=file:///tmp/pitch_range_180/GripperDragonWithServo_urdf_mes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
Joints:
- removed joint bone_2_to_endeffector
- removed joint joint_2_to_bone_2
- added joint endeffector_to_dummy_object: type revolute, parent endeffector, child dummy_object_link, origin xyz=0 0 147 rpy=0 0 0, axis 1 0 0, limit lower=0 upper=0 effort=1.0 velocity=1.0
- added joint joint_2_to_endeffector: type revolute, parent joint_2, child endeffector, origin xyz=0 0 200 rpy=0 0 0, axis 1 0 0, limit lower=-1.48353 upper=1.48353 effort=1.0 velocity=1.0

File: urdf/ato_3_seg_270_deg.urdf (robot description, URDF)
Before this commit: robot ato, 8 links, 7 joints
Links:
- removed link bone_3
- removed link endeffector_link
- added link dummy_object_link; visual box size=1 2 3
- added link endeffector; visual mesh filename=file:///tmp/pitch_range_270/GripperDragonWithServo_urdf_mes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
Joints:
- removed joint bone_3_to_endeffector
- removed joint joint_3_to_bone_3
- added joint endeffector_to_dummy_object: type revolute, parent endeffector, child dummy_object_link, origin xyz=0 0 147 rpy=0 0 0, axis 1 0 0, limit lower=0 upper=0 effort=1.0 velocity=1.0
- added joint joint_3_to_endeffector: type revolute, parent joint_3, child endeffector, origin xyz=0 0 220 rpy=0 0 0, axis 1 0 0, limit lower=-2.26893 upper=2.26893 effort=1.0 velocity=1.0

Commit message: Added pibullet visualization
Tuned cartesian control

To debug pitch issue at negative angles (upwards)

File: urdf/ato_2_seg_180_deg.urdf (robot description, URDF)
Before this commit: robot ato, 6 links, 5 joints
Links:
- removed link base_link
- added link bone_0, mass 0.0; visual mesh filename=file:///tmp/pitch_range_180/BoneAugmented_urdf_mesh.stl
Joints:
- removed joint base_link_to_joint_1
- added joint bone_0_to_joint_1: type revolute, parent bone_0, child joint_1, origin xyz=0 0 0 rpy=0 0 0, axis 0 0 1, limit lower=-1.5708 upper=1.5708 effort=1.0 velocity=1.0

File: urdf/ato_3_seg_270_deg.urdf (robot description, URDF)
Before this commit: robot ato, 8 links, 7 joints
Links:
- removed link base_link
- added link bone_0, mass 0.0; visual mesh filename=file:///tmp/pitch_range_270/BoneAugmented_urdf_mesh.stl
Joints:
- removed joint base_link_to_joint_1
- added joint bone_0_to_joint_1: type revolute, parent bone_0, child joint_1, origin xyz=0 0 0 rpy=0 0 0, axis 0 0 1, limit lower=-2.35619 upper=2.35619 effort=1.0 velocity=1.0
